Commit message: loads amiga with ur5e in new base config

File: trajectory_cache/urdf/ur5e/ur5e.urdf (robot description, URDF)
Before this commit: robot ur5e, 12 links, 11 joints
Links:
- added link gripper_body_link; collision box size=0.12 0.12 0.2; visual box size=0.12 0.12 0.2
- link gripper_link: geometry 
Joints:
- added joint eef_joint: type fixed, parent gripper_body_link, child gripper_link, origin xyz=0 0 0 rpy=0 0 0
- joint gripper_joint: child gripper_link -> gripper_body_link

Commit message: Loads amiga stl and adds collision objs for other items present in amiga urdf

File: trajectory_cache/urdf/ur5e/ur5e.urdf (robot description, URDF)
Before this commit: robot ur5e, 13 links, 12 joints
Joints:
- joint eef_joint: origin xyz=0 0 0 rpy=0 0 0 -> xyz=0 0 0.105 rpy=0 0 0
- joint gripper_joint: origin xyz=0 0 0.215 rpy=0 0 0 -> xyz=0 0 0.105 rpy=0 0 0
