Commit message: adds end-effector stl

File: trajectory_cache/urdf/ur5e/ur5e.urdf (robot description, URDF)
Before this commit: robot ur5e, 13 links, 12 joints
Links:
- added link hose_mount_clip_link; collision box size=0.02 0.025 0.02; visual box size=0.02 0.025 0.02
- link gripper_body_link: geometry collision mesh filename=../end-effector/Finray2526-URDF-Collision.stl scale=0.001 0.001 0.001; visual mesh filename=../end-effector/Finray2526-URDF-Collision.stl scale=0.001 0.001 0.001
Joints:
- added joint hose_mount_joint: type fixed, parent tool0, child hose_mount_clip_link, origin xyz=0.05 0 -0.025 rpy=0 0 0
- joint eef_joint: origin xyz=0 0 0.105 rpy=0 0 0 -> xyz=0 0 0.29 rpy=0 0 0
- joint gripper_joint: origin xyz=0 0 0.105 rpy=0 0 0 -> xyz=0 0 0 rpy=0 0 3.14159

Commit message: updates link geometry to better mesh with the hybrid planner

File: trajectory_cache/urdf/ur5e/ur5e.urdf (robot description, URDF)
Before this commit: robot ur5e, 14 links, 13 joints
Joints:
- joint gripper_joint: origin xyz=0 0 0 rpy=0 0 3.14159 -> xyz=0 0 0 rpy=0 0 0
